Commit message: solve ik

File: examples/robots/fetch/fetch.urdf (robot description, URDF)
Before this commit: robot fetch, 26 links, 25 joints
Joints:
- joint forearm_roll_joint: limit effort=29.35 velocity=1.571 -> lower=-3.14 upper=3.14 effort=29.35 velocity=1.571
- joint upperarm_roll_joint: limit effort=76.94 velocity=1.571 -> lower=-3.14 upper=3.14 effort=76.94 velocity=1.571
- joint wrist_roll_joint: limit effort=7.36 velocity=2.268 -> lower=-3.14 upper=3.14 effort=7.36 velocity=2.268
