Commit message: test grasping

File: examples/objects/cafe_table/cafe_table.urdf (robot description, URDF)
Before this commit: robot cafe_table_org, 1 links, 0 joints
Links:
- link baseLink: mass 1.0 -> 100.0

Commit message: test grasping

File: examples/objects/cafe_table/cafe_table.urdf (robot description, URDF)
Before this commit: robot cafe_table_org, 1 links, 0 joints
Links:
- link baseLink: mass 1.0 -> 0.0

Commit message: change table mass to 0

File: examples/objects/cafe_table/cafe_table.urdf (robot description, URDF)
Before this commit: robot cafe_table_org, 1 links, 0 joints
Links:
- link baseLink: mass 100.0 -> 0
