Commit message: use panda with camera

File: examples/robots/panda/panda.urdf (robot description, URDF)
Before this commit: robot panda, 12 links, 11 joints
Links:
- removed link panda_link8
- added link panda_hand_camera, mass 0.01; collision mesh filename=meshes/collision/camera.stl; visual mesh filename=meshes/visual/camera.obj
- link panda_hand: mass None -> 0.68; geometry collision mesh filename=meshes/collision/hand.obj; visual mesh filename=meshes/visual/hand.obj
- link panda_leftfinger: mass None -> 0.01; geometry collision mesh filename=meshes/collision/finger.obj; visual mesh filename=meshes/visual/finger.obj
- link panda_link0: mass None -> 3.06; geometry collision mesh filename=meshes/collision/link0.obj; visual mesh filename=meshes/collision/link0.obj
- link panda_link1: mass None -> 2.34; geometry collision mesh filename=meshes/collision/link1.obj; visual mesh filename=meshes/visual/link1.obj
- link panda_link2: mass None -> 2.36; geometry collision mesh filename=meshes/collision/link2.obj; visual mesh filename=meshes/visual/link2.obj
- link panda_link3: mass None -> 2.38; geometry collision mesh filename=meshes/collision/link3.obj; visual mesh filename=meshes/visual/link3.obj
- link panda_link4: mass None -> 2.43; geometry collision mesh filename=meshes/collision/link4.obj; visual mesh filename=meshes/visual/link4.obj
- link panda_link5: mass None -> 3.5; geometry collision mesh filename=meshes/collision/link5.obj; visual mesh filename=meshes/visual/link5.obj
- link panda_link6: mass None -> 1.47; geometry collision mesh filename=meshes/collision/link6.obj; visual mesh filename=meshes/visual/link6.obj
- link panda_link7: mass None -> 0.45; geometry collision mesh filename=meshes/collision/link7.obj; visual mesh filename=meshes/collision/link7.obj
- link panda_rightfinger: mass None -> 0.01; geometry collision mesh filename=meshes/collision/finger.obj; visual mesh filename=meshes/visual/finger.obj
Joints:
- removed joint panda_joint8
- added joint panda_hand_camera_joint: type fixed, parent panda_hand, child panda_hand_camera, origin xyz=0.036 0 0.036 rpy=-1.57079632679 0 -1.57079632679
- joint panda_hand_joint: origin xyz=0 0 0 rpy=0 0 -0.785398163397 -> xyz=0 0 0.107 rpy=0 0 -0.785398163397; parent panda_link8 -> panda_link7
- joint panda_joint6: limit lower=-0.0175 upper=3.7525 effort=12 velocity=2.6100 -> lower=-0.0175 upper=3.752 effort=12 velocity=2.6100

File: examples/robots/panda/panda_gripper.urdf (robot description, URDF)
Before this commit: robot panda_gripper, 3 links, 2 joints
Links:
- added link panda_hand_camera, mass 0.01; collision mesh filename=meshes/collision/camera.stl; visual mesh filename=meshes/visual/camera.obj
- link panda_hand: mass None -> 0.68; geometry collision mesh filename=meshes/collision/hand.obj; visual mesh filename=meshes/visual/hand.obj
- link panda_leftfinger: mass None -> 0.01; geometry collision mesh filename=meshes/collision/finger.obj; visual mesh filename=meshes/visual/finger.obj
- link panda_rightfinger: mass None -> 0.01; geometry collision mesh filename=meshes/collision/finger.obj; visual mesh filename=meshes/visual/finger.obj
Joints:
- added joint panda_hand_camera_joint: type fixed, parent panda_hand, child panda_hand_camera, origin xyz=0.036 0 0.036 rpy=-1.57079632679 0 -1.57079632679

Commit message: fix panda urdf

File: examples/robots/panda/panda.urdf (robot description, URDF)
Before this commit: robot panda, 12 links, 11 joints
Links:
- link panda_hand: geometry collision mesh filename=meshes/collision/hand.stl; visual mesh filename=meshes/visual/hand.obj
- link panda_leftfinger: geometry collision mesh filename=meshes/collision/finger.stl; visual mesh filename=meshes/visual/finger.obj
- link panda_link0: geometry collision mesh filename=meshes/collision/link0.stl; visual mesh filename=meshes/visual/link0.obj
- link panda_link1: geometry collision mesh filename=meshes/collision/link1.stl; visual mesh filename=meshes/visual/link1.obj
- link panda_link2: geometry collision mesh filename=meshes/collision/link2.stl; visual mesh filename=meshes/visual/link2.obj
- link panda_link3: geometry collision mesh filename=meshes/collision/link3.stl; visual mesh filename=meshes/visual/link3.obj
- link panda_link4: geometry collision mesh filename=meshes/collision/link4.stl; visual mesh filename=meshes/visual/link4.obj
- link panda_link5: geometry collision mesh filename=meshes/collision/link5.stl; visual mesh filename=meshes/visual/link5.obj
- link panda_link6: geometry collision mesh filename=meshes/collision/link6.stl; visual mesh filename=meshes/visual/link6.obj
- link panda_link7: geometry collision mesh filename=meshes/collision/link7.stl; visual mesh filename=meshes/visual/link7.obj
- link panda_rightfinger: geometry collision mesh filename=meshes/collision/finger.stl; visual mesh filename=meshes/visual/finger.obj

File: examples/robots/panda/panda_gripper.urdf (robot description, URDF)
Before this commit: robot panda_gripper, 4 links, 3 joints
Links:
- link panda_hand: geometry collision mesh filename=meshes/collision/hand.stl; visual mesh filename=meshes/visual/hand.obj
- link panda_leftfinger: geometry collision mesh filename=meshes/collision/finger.stl; visual mesh filename=meshes/visual/finger.obj
- link panda_rightfinger: geometry collision mesh filename=meshes/collision/finger.stl; visual mesh filename=meshes/visual/finger.obj
