Commit message: use fetch igibson

File: data/robots/fetch_igibson/fetch.urdf (robot description, URDF)
Before this commit: robot fetch, 24 links, 23 joints
Links:
- added link l_gripper_finger_link, mass 0.0798; collision mesh filename=meshes/l_gripper_finger_link.obj; visual mesh filename=meshes/l_gripper_finger_link.obj
- added link r_gripper_finger_link, mass 0.0798; collision mesh filename=meshes/r_gripper_finger_link.obj; visual mesh filename=meshes/r_gripper_finger_link.obj
Joints:
- added joint l_gripper_finger_joint: type prismatic, parent gripper_link, child l_gripper_finger_link, origin xyz=0 -0.015425 0 rpy=0 0 0, axis 0 -1 0, limit lower=0.0 upper=0.05 effort=60 velocity=0.05
- added joint r_gripper_finger_joint: type prismatic, parent gripper_link, child r_gripper_finger_link, origin xyz=0 0.015425 0 rpy=0 0 0, axis 0 1 0, limit lower=0.0 upper=0.05 effort=60 velocity=0.05
- joint eye_joint: parent head_camera_depth_frame -> head_camera_link
- joint forearm_roll_joint: limit effort=29.35 velocity=1.571 -> lower=-3.14 upper=3.14 effort=29.35 velocity=1.571
- joint head_pan_joint: type fixed -> revolute
- joint head_tilt_joint: origin xyz=0.14253 0 0.057999 rpy=0 0.17453292519943295 0 -> xyz=0.14253 0 0.057999 rpy=0 0.2617993877991494 0; type fixed -> revolute
- joint upperarm_roll_joint: limit effort=76.94 velocity=1.571 -> lower=-3.14 upper=3.14 effort=76.94 velocity=1.571
- joint wrist_roll_joint: limit effort=7.36 velocity=2.268 -> lower=-3.14 upper=3.14 effort=7.36 velocity=2.268

File: data/robots/fetch_igibson/fetch_gripper.urdf (robot description, URDF)
Before this commit: robot fetch, 26 links, 25 joints
Links:
- removed link base_link
- removed link caster_wheel_link
- removed link elbow_flex_link
- removed link estop_link
- removed link eyes
- removed link forearm_roll_link
- removed link head_camera_depth_frame
- removed link head_camera_depth_optical_frame
- removed link head_camera_link
- removed link head_camera_rgb_frame
- removed link head_camera_rgb_optical_frame
- removed link head_pan_link
- removed link head_tilt_link
- removed link l_wheel_link
- removed link laser_link
- removed link r_wheel_link
- removed link shoulder_lift_link
- removed link shoulder_pan_link
- removed link torso_fixed_link
- removed link torso_lift_link
- removed link upperarm_roll_link
- removed link wrist_flex_link
Joints:
- removed joint caster_wheel_joint
- removed joint elbow_flex_joint
- removed joint estop_joint
- removed joint eye_joint
- removed joint forearm_roll_joint
- removed joint head_camera_depth_joint
- removed joint head_camera_depth_optical_joint
- removed joint head_camera_joint
- removed joint head_camera_rgb_joint
- removed joint head_camera_rgb_optical_joint
- removed joint head_pan_joint
- removed joint head_tilt_joint
- removed joint l_wheel_joint
- removed joint laser_joint
- removed joint r_wheel_joint
- removed joint shoulder_lift_joint
- removed joint shoulder_pan_joint
- removed joint torso_fixed_joint
- removed joint torso_lift_joint
- removed joint upperarm_roll_joint
- removed joint wrist_flex_joint
- removed joint wrist_roll_joint
